File: KiCadV2/PerCoil.kicad_sch (KiCad schematic)
At the start: 15 parts, among them U20 DMHT10H032LFJ, U21 INA240A1D

Commit message: idk
Parts:
- removed C18: 100n, Capacitor_SMD:C_0603_1608Metric, symbol Device:C
- removed C19: 2.2u, Capacitor_SMD:C_0603_1608Metric, symbol Device:C
- removed R25, R26: 2k, Resistor_SMD:R_0603_1608Metric, symbol Device:R
- C17: renamed from C20; LCSC (none) -> C14663
- C18: renamed from C21; LCSC (none) -> C14663
- D9: footprint Diode_SMD:D_SMA -> Diode_SMD:D_SOD-323; LCSC (none) -> C7420329
- R24: renamed from R27; LCSC (none) -> C42460614
- R25: renamed from R28; LCSC (none) -> C42460614
- R27: renamed from R30; LCSC (none) -> C21190
- R28: renamed from R31; LCSC (none) -> C21190
- U18: renamed from U20; now left out of the parts list
- U19: renamed from U21; LCSC (none) -> C2060769
- renumbered R29 to R26

Commit message: schematic FINAL! (I hope)
Parts:
- added D8: KT-0603W, LED_SMD:LED_0603_1608Metric, symbol Device:LED
- added R16: 12k, Resistor_SMD:R_0603_1608Metric, symbol Device:R
- added R17: 10k, Resistor_SMD:R_0603_1608Metric, symbol Device:R
- added R18: 100, Resistor_SMD:R_0603_1608Metric, symbol Device:R
- added R19: 390, Resistor_SMD:R_0603_1608Metric, symbol Device:R
- added U14: 74LV08AT14-13, Package_SO:TSSOP-14_4.4x5mm_P0.65mm, symbol 74xx:74LV08AT14-13
- added U18: MX3502S, Package_SO:SOP-8_3.76x4.96mm_P1.27mm, symbol Comparator:MX3502
- added U20, U21: ~, TestPoint:SPDT_solder_bridge, symbol Connector:SPDT_solder_bridge
- L2: footprint Inductor_SMD:L_TDK_SLF12555 -> Inductor_SMD:6.8uH C5127257
- renumbered C18 to C15, C17 to C16, R24 to R20, R25 to R21, R26 to R22, R27 to R23, R28 to R24, U18 to U22, U19 to U23
Connections:
- net +5V: now also R19.2, U14.12 (B)
- net Analog_Sense: now also U20.1 (A), U21.1 (A)
- net EN: now also R17.1, U14.8 (A)
- net GND: now also R17.2
- net OC_SENSE: now also U18.4 (-)
- net VCM_HIGHZ: now also U20.3 (B), U21.3 (B)
- net VBUS renamed Vdrive
- new net: U18.1 (+), U20.2 (COM)
- new net: R16.1, R18.2, U18.3 (+)
- new net: U18.2 (-), U21.2 (COM)
- new net: D8.2 (A), R19.1
- new net: D8.1 (K), U14.13 (Y)
- new net 0.2V: R18.1
- new net SignalProcessingChain/Current_Dir: U18.7
- new net SignalProcessingChain/EN: U14.10 (Y)
- new net ~{OC1}: R16.2, U14.11 (A), U14.9 (B), U18.6
Other:
- sheet SignalProcessingChain ports: added Current_Dir, Vtri; removed none
- note added: "0.1ohm current sense resistor"
- note added: "20V/V Diff amp w/ strong common-mode rejection, and like +/- 60V or smt common-mode operating region."
- note added: "AND gate for external EN pin"
- note added: "Buffer"
- note added: "Chain of muxes, gates, etc that determine which signals go where depending on mode bits A,B,C,EN. Also includes ~1MHz PWM upscaler."
- note added: "Current sense"
- note added: "H-bridge"
- note added: "If OC, EN forced low by this comparator"
- note added: "Indicator LED"
- note added: "LPF to remove current ripple Also includes divider to set LF gain, so diff-amp output doesn't saturate."
- note added: "OC_SENSE must stay within -0.3V to 5.3V, or else comparator in OC detection will be damaged. Shottkey protects this. (5.3V not possible, since that would imply 53A and the whole board would have exploded long before then)"
- note added: "One more LPF to remove any noise or ripple"
- note added: "Over-current (OC) detection"
- note added: "Set DIR to whichever direction the current is traveling"
- note removed: "Current sense: RC LPF to remove current ripple -> 20V/V diff amp"
- moved on the sheet: C15, C16, D9, L2, R20, R21, R22, R23, R24, U22, U23

Commit message: PCB Almost done with one coil!!
Parts:
- added C30, C47: 100n, Capacitor_SMD:C_0603_1608Metric, symbol Device:C
Connections:
- net +5V: now also C47.1
- net 0.2V: now also C30.2
- net GND: now also C30.1, C47.2
- net OC_SENSE: now also U18.2 (-); no longer U18.4 (-)
- net SignalProcessingChain/Current_Dir: now also U18.6; no longer U18.7
- net ~{OC1}: now also U18.7; no longer U18.6
- net at U20.2 (COM): now also U18.3 (+); no longer U18.1 (+)
- net at R16.1, R18.2: now also U18.1 (+); no longer U18.3 (+)
- net at U21.2 (COM): now also U18.4 (-); no longer U18.2 (-)
Other:
- note added: "Decoupling cap"
