File: KiCadV2/untitled.kicad_sch (KiCad schematic)
At the start: 13 parts, among them U32 MCP6002-xSN, U33 CJ432

Commit message: idk
Parts:
- removed C40, C42: 100n, Capacitor_SMD:C_0603_1608Metric, symbol Device:C
- C33: renamed from C41; LCSC (none) -> C23630
- C34: renamed from C43; LCSC (none) -> C23630
- R43: renamed from R49; value 250 -> 200; footprint Resistor_SMD:R_0603_1608Metric -> Resistor_SMD:R_0805_2012Metric; LCSC (none) -> C17540
- R44: renamed from R50; LCSC (none) -> C25804
- R45: renamed from R51; LCSC (none) -> C25804
- R46: renamed from R52; value 9200 -> 9.1k; LCSC (none) -> C23260
- R47: renamed from R53; value 800 -> 820; LCSC (none) -> C23253
- R48: renamed from R54; LCSC (none) -> C22775
- R49: renamed from R55; LCSC (none) -> C22775
- U29: renamed from U32; LCSC (none) -> C7377
- U30: renamed from U33; LCSC (none) -> C3113
Connections:
- net at U29.1, U29.2 (-): now also R48.1
Other:
- note added: "~20mA"

Commit message: schematic FINAL! (I hope)
Parts:
- renumbered C33 to C29, C34 to C30, R43 to R40, R44 to R41, R45 to R42, R46 to R43, R47 to R44, R48 to R45, R49 to R46, U29 to U40, U30 to U41
Changed lines of the file:
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@@
 		(dnp no)
 		(fields_autoplaced yes)
-		(property "Reference" "U29"
+		(property "Reference" "U40"
 			(at 83.82 95.2499 0)
 			(effects
@@
 			(project "KiCadV2"
 				(path "/e7727714-8b02-4dc5-9ae4-9abf282a37e0/119d2b89-5afc-44da-b120-a3e681adcba0"
-					(reference "U29")
+					(reference "U40")
 					(unit 3)
 				)
@@
 		(dnp no)
 		(fields_autoplaced yes)
-		(property "Reference" "R44"
+		(property "Reference" "R41"
 			(at 114.3 63.4999 0)
 			(effects
@@
 			(project "KiCadV2"
 				(path "/e7727714-8b02-4dc5-9ae4-9abf282a37e0/119d2b89-5afc-44da-b120-a3e681adcba0"
-					(reference "R44")
+					(reference "R41")
 					(unit 1)
 				)
@@
 		(dnp no)
 		(fields_autoplaced yes)
-		(property "Reference" "U30"
+		(property "Reference" "U41"
 			(at 113.03 129.5399 90)
 			(effects
@@
 			(project "KiCadV2"
 				(path "/e7727714-8b02-4dc5-9ae4-9abf282a37e0/119d2b89-5afc-44da-b120-a3e681adcba0"
-					(reference "U30")
+					(reference "U41")
 					(unit 1)
 				)
@@
 		(dnp no)
 		(fields_autoplaced yes)
-		(property "Reference" "R47"
+		(property "Reference" "R44"
 			(at 124.46 130.8099 0)
 			(effects
@@
 			(project "KiCadV2"
 				(path "/e7727714-8b02-4dc5-9ae4-9abf282a37e0/119d2b89-5afc-44da-b120-a3e681adcba0"
-					(reference "R47")
+					(reference "R44")
 					(unit 1)
 				)
@@
 		(dnp no)
 		(fields_autoplaced yes)
-		(property "Reference" "R45"
+		(property "Reference" "R42"
 			(at 114.3 78.7399 0)
 			(effects
@@
 			(project "KiCadV2"
 				(path "/e7727714-8b02-4dc5-9ae4-9abf282a37e0/119d2b89-5afc-44da-b120-a3e681adcba0"
-					(reference "R45")
+					(reference "R42")
 					(unit 1)
 				)
@@
 		(dnp no)
 		(fields_autoplaced yes)
-		(property "Reference" "R43"
+		(property "Reference" "R40"
 			(at 113.03 111.7599 0)
 			(effects
@@
 			(project "KiCadV2"
 				(path "/e7727714-8b02-4dc5-9ae4-9abf282a37e0/119d2b89-5afc-44da-b120-a3e681adcba0"
-					(reference "R43")
+					(reference "R40")
 					(unit 1)
 				)
@@
 		(dnp no)
 		(fields_autoplaced yes)
-		(property "Reference" "R49"
+		(property "Reference" "R46"
 			(at 148.59 123.19 90)
 			(effects
@@
 			(project "KiCadV2"
 				(path "/e7727714-8b02-4dc5-9ae4-9abf282a37e0/119d2b89-5afc-44da-b120-a3e681adcba0"
-					(reference "R49")
+					(reference "R46")
 					(unit 1)
 				)
@@
 		(dnp no)
 		(fields_autoplaced yes)
-		(property "Reference" "R46"
+		(property "Reference" "R43"
 			(at 124.46 120.6499 0)
 			(effects
@@
 			(project "KiCadV2"
 				(path "/e7727714-8b02-4dc5-9ae4-9abf282a37e0/119d2b89-5afc-44da-b120-a3e681adcba0"
-					(reference "R46")
+					(reference "R43")
 					(unit 1)
 				)
@@
 		(dnp no)
 		(fields_autoplaced yes)
-		(property "Reference" "U29"
+		(property "Reference" "U40"
 			(at 127 64.77 0)
 			(effects
@@
 			(project "KiCadV2"
 				(path "/e7727714-8b02-4dc5-9ae4-9abf282a37e0/119d2b89-5afc-44da-b120-a3e681adcba0"
-					(reference "U29")
+					(reference "U40")
 					(unit 1)
 				)
@@
 		(dnp no)
 		(fields_autoplaced yes)
-		(property "Reference" "C33"
+		(property "Reference" "C29"
 			(at 157.48 77.4699 0)
 			(effects
@@
 			(project "KiCadV2"
 				(path "/e7727714-8b02-4dc5-9ae4-9abf282a37e0/119d2b89-5afc-44da-b120-a3e681adcba0"
-					(reference "C33")
+					(reference "C29")
 					(unit 1)
 				)
@@
 		(dnp no)
 		(fields_autoplaced yes)
-		(property "Reference" "C34"
+		(property "Reference" "C30"
 			(at 165.1 132.0799 0)
 			(effects
@@
 			(project "KiCadV2"
 				(path "/e7727714-8b02-4dc5-9ae4-9abf282a37e0/119d2b89-5afc-44da-b120-a3e681adcba0"
-					(reference "C34")
+					(reference "C30")
 					(unit 1)
 				)
@@
 		(dnp no)
 		(fields_autoplaced yes)
-		(property "Reference" "R48"
+		(property "Reference" "R45"
 			(at 139.7 68.58 90)
 			(effects
@@
 			(project "KiCadV2"
 				(path "/e7727714-8b02-4dc5-9ae4-9abf282a37e0/119d2b89-5afc-44da-b120-a3e681adcba0"
-					(reference "R48")
+					(reference "R45")
 					(unit 1)
 				)
@@
 		(dnp no)
 		(fields_autoplaced yes)
-		(property "Reference" "U29"
+		(property "Reference" "U40"
 			(at 137.16 119.38 0)
 			(effects
@@
 			(project "KiCadV2"
 				(path "/e7727714-8b02-4dc5-9ae4-9abf282a37e0/119d2b89-5afc-44da-b120-a3e681adcba0"
-					(reference "U29")
+					(reference "U40")
 					(unit 2)
 				)

Commit message: PCB Almost done with one coil!!
Parts:
- removed C30: 2.2u, Capacitor_SMD:C_0603_1608Metric, symbol Device:C
Changed lines of the file:
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@@
-	)
-	(junction
-		(at 161.29 129.54)
-		(diameter 0)
-		(color 0 0 0 0)
 	)
 	(junction
@@
 		(color 0 0 0 0)
 	)
-	(junction
-		(at 157.48 137.16)
-		(diameter 0)
-		(color 0 0 0 0)
-	)
 	(wire
 		(pts
@@
 	(wire
 		(pts
-			(xy 153.67 137.16) (xy 157.48 137.16)
-		)
-		(stroke
-			(width 0)
-			(type default)
-		)
-	)
-	(wire
-		(pts
-			(xy 152.4 129.54) (xy 161.29 129.54)
+			(xy 152.4 129.54) (xy 165.1 129.54)
 		)
 		(stroke
@@
 	(wire
 		(pts
-			(xy 161.29 129.54) (xy 165.1 129.54)
-		)
-		(stroke
-			(width 0)
-			(type default)
-		)
-	)
-	(wire
-		(pts
 			(xy 119.38 81.28) (xy 134.62 81.28)
 		)
@@
 		(pts
 			(xy 111.76 68.58) (xy 111.76 72.39)
-		)
-		(stroke
-			(width 0)
-			(type default)
-		)
-	)
-	(wire
-		(pts
-			(xy 157.48 137.16) (xy 161.29 137.16)
 		)
 		(stroke
@@
 	)
 	(symbol
-		(lib_id "power:GND")
-		(at 157.48 137.16 0)
-		(unit 1)
-		(exclude_from_sim no)
-		(in_bom yes)
-		(on_board yes)
-		(dnp no)
-		(fields_autoplaced yes)
-		(property "Reference" "#PWR0102"
-			(at 157.48 143.51 0)
-			(effects
-				(font
-					(size 1.27 1.27)
-				)
-				(hide yes)
-			)
-		)
-		(property "Value" "GND"
-			(at 157.48 142.24 0)
-			(effects
-				(font
-					(size 1.27 1.27)
-				)
-			)
-		)
-		(property "Footprint" ""
-			(at 157.48 137.16 0)
-			(effects
-				(font
-					(size 1.27 1.27)
-				)
-				(hide yes)
-			)
-		)
-		(property "Datasheet" ""
-			(at 157.48 137.16 0)
-			(effects
-				(font
-					(size 1.27 1.27)
-				)
-				(hide yes)
-			)
-		)
-		(property "Description" "Power symbol creates a global label with name \"GND\" , ground"
-			(at 157.48 137.16 0)
-			(effects
-				(font
-					(size 1.27 1.27)
-				)
-				(hide yes)
-			)
-		)
-		(pin "1"
-		)
-		(instances
-			(project "KiCadV2"
-				(path "/e7727714-8b02-4dc5-9ae4-9abf282a37e0/119d2b89-5afc-44da-b120-a3e681adcba0"
-					(reference "#PWR0102")
-					(unit 1)
-				)
-			)
-		)
-	)
-	(symbol
 		(lib_id "Device:R")
 		(at 111.76 64.77 0)
@@
 					(unit 1)
 				)
-			)
-		)
-	)
-	(symbol
-		(lib_id "Device:C")
-		(at 161.29 133.35 180)
-		(unit 1)
-		(exclude_from_sim no)
-		(in_bom yes)
-		(on_board yes)
-		(dnp no)
-		(fields_autoplaced yes)
-		(property "Reference" "C30"
-			(at 165.1 132.0799 0)
-			(effects
-				(font
-					(size 1.27 1.27)
-				)
-				(justify right)
-			)
-		)
-		(property "Value" "2.2u"
-			(at 165.1 134.6199 0)
-			(effects
-				(font
-					(size 1.27 1.27)
-				)
-				(justify right)
-			)
-		)
-		(property "Footprint" "Capacitor_SMD:C_0603_1608Metric"
-			(at 160.3248 129.54 0)
-			(effects
-				(font
-					(size 1.27 1.27)
-				)
-				(hide yes)
-			)
-		)
-		(property "Datasheet" "~"
-			(at 161.29 133.35 0)
-			(effects
-				(font
-					(size 1.27 1.27)
-				)
-				(hide yes)
-			)
-		)
-		(property "Description" "Unpolarized capacitor"
-			(at 161.29 133.35 0)
-			(effects
-				(font
-					(size 1.27 1.27)
-				)
-				(hide yes)
-			)
-		)
-		(property "LCSC" "C23630"
-			(at 161.29 133.35 0)
-			(effects
-				(font
-					(size 1.27 1.27)
-				)
-				(hide yes)
-			)
-		)
-		(pin "1"
-		)
-		(pin "2"
-		)
-		(instances
-			(project "KiCadV2"
-				(path "/e7727714-8b02-4dc5-9ae4-9abf282a37e0/119d2b89-5afc-44da-b120-a3e681adcba0"
-					(reference "C30")
-					(unit 1)
-				)
