File: KiCadV2/PerCoilFlipped.kicad_sch (KiCad schematic)
At the start: 22 parts, among them U14 74LV08AT14-13, U18 MX3502S, U22 DMHT10H032LFJ, U23 INA240A1D

Commit message: saving here before i try making PerCoilFlipped on schematic
Parts:
- renumbered C15 to C17, C16 to C18, C47 to C48, C30 to C49, D8 to D10, D9 to D11, L2 to L3, R16 to R25, R17 to R26, R18 to R27, R19 to R28, R20 to R29, R21 to R30, R22 to R31, R23 to R32, R24 to R33, U18 to U26, U20 to U28, U21 to U29, U22 to U30, U23 to U31, U14 to U38
Connections:
- net AH: now also U30.10 (G4); no longer U30.1 (G1)
- net AL: now also U30.7 (G3); no longer U30.4 (G2)
- net BH: now also U30.1 (G1); no longer U30.10 (G4)
- net BHS: now also U30.3 (S1/D2); no longer U30.8 (S4/D3)
- net BL: now also U30.4 (G2); no longer U30.7 (G3)
- net COIL+: now also U30.8 (S4/D3); no longer U30.3 (S1/D2)
Other:
- moved on the sheet: U30
