File: KiCadV2/SignalProcessingChain.kicad_sch (KiCad schematic)
At the start: 35 parts, among them U19 HIP4080A

Commit message: idk
Parts:
- removed C12, C13: 100n, Capacitor_SMD:C_0603_1608Metric, symbol Device:C
- removed D6: D, Diode_SMD:D_SMA, symbol Device:D
- removed R21: 10k, Resistor_SMD:R_0603_1608Metric, symbol Device:R
- removed U16: ~, Package_TO_SOT_SMD:SOT-363_SC-70-6, symbol 74xx:NC7SZ157P6X
- added U6: 74LV08AT14-13, Package_SO:TSSOP-14_4.4x5mm_P0.65mm, symbol 74xx:74LV08AT14-13
- added U9: GT74LVC6G14TD, Package_SO:TSSOP-14_4.4x5mm_P0.65mm, symbol 74xx:74HC04
- C10: renamed from C9; LCSC C1620 -> C396711
- C13: renamed from C15; LCSC (none) -> C14663
- C15: renamed from C16; value 1uF -> 100n; LCSC (none) -> C14663
- C16: renamed from C17; value 1uF -> 100n; LCSC (none) -> C14663
- C6: renamed from C5; value C -> 33n; LCSC (none) -> C21117
- D7, D8: value D -> D_bootstrap; footprint Diode_SMD:D_SMA -> Diode_SMD:D_SOD-523; LCSC (none) -> C7502714
- R15: value R -> 2700; LCSC (none) -> C13167
- R16: value R -> 1500; LCSC (none) -> C22843
- R17: value R -> 2000; LCSC (none) -> C22975
- R22: renamed from R23; value 50k -> 51k; LCSC (none) -> C23196
- R23: renamed from R24; value 50k -> 51k; LCSC (none) -> C23196
- U11: renamed from U12; value ~ -> MX3502S
- U12: renamed from U13; value ~ -> NC7SZ157P6X
- U13: renamed from U14; value ~ -> NC7SZ157P6X
- U14: renamed from U15; value ~ -> NC7SZ157P6X
- U15: renamed from U17; value ~ -> NC7SZ157P6X
- U16: renamed from U18; value ~ -> NC7SZ157P6X
- U17: renamed from U19; now left out of the parts list
- renumbered C10 to C11, C11 to C12, C4 to C5, C6 to C7, C7 to C8, C8 to C9, R22 to R21
Connections:
- net +5V: no longer C14.1
- net C: now also U6.9 (B)
- net EN: now also U6.8 (A), U9.5
- net EN*C: now also U6.10 (Y)
- net VCM_HIGHZ: now also C14.1
- net Vtri: now also C10.1, R20.1, U11.2 (-); no longer R18.2, R19.1, U11.1 (+)
- net at U16.3 (I0): now also U9.6
- new net: R18.2, R19.1, U11.1 (+)
Other:
- note removed: "1x Inv"
- note removed: "EN*C AND"

Commit message: schematic FINAL! (I hope)
Parts:
- removed C10: 470p, Capacitor_SMD:C_0603_1608Metric, symbol Device:C
- removed C5, C7: 100n, Capacitor_SMD:C_0603_1608Metric, symbol Device:C
- removed C8: 2.2u, Capacitor_SMD:C_0603_1608Metric, symbol Device:C
- removed R18: 1k, Resistor_SMD:R_0603_1608Metric, symbol Device:R
- removed R19: 9.1k, Resistor_SMD:R_0603_1608Metric, symbol Device:R
- removed R20: 5.1k, Resistor_SMD:R_0603_1608Metric, symbol Device:R
- removed unit 3 of U11
- removed unit 1 of U11
- removed U6: 74LV08AT14-13, Package_SO:TSSOP-14_4.4x5mm_P0.65mm, symbol 74xx:74LV08AT14-13
- removed U9: GT74LVC6G14TD, Package_SO:TSSOP-14_4.4x5mm_P0.65mm, symbol 74xx:74HC04
- added C43, C45, C6: 100n, Capacitor_SMD:C_0603_1608Metric, symbol Device:C
- added TP2: TestPoint, TestPoint:TestPoint_Pad_D2.5mm, symbol Connector:TestPoint
- added U10: NC7SZ157P6X, Package_TO_SOT_SMD:SOT-363_SC-70-6, symbol 74xx:NC7SZ157P6X
- added U14: 74LV08AT14-13, Package_SO:TSSOP-14_4.4x5mm_P0.65mm, symbol 74xx:74LV08AT14-13
- renumbered C12 to C10, C13 to C11, C14 to C12, C15 to C13, C16 to C14, C6 to C5, C9 to C8, C11 to C9, D7 to D6, D8 to D7, R15 to R10, R16 to R11, R17 to R12, R22 to R13, R23 to R14, R21 to R15, U14 to U11, U15 to U12, U16 to U13, U17 to U15, U11 to U17, U12 to U8, U13 to U9
Connections:
- net EN*C is gone; now on net C: U13.6 (S)
- net +5V: now also C43.1, C45.1, C6.1, U10.5 (Vcc)
- net DIR: now also U10.4 (Z); no longer U9.4 (Z)
- net DIS: now also U14.6 (Y); no longer U13.4 (Z)
- net EN: now also U10.6 (S), U14.2 (B), U14.4 (A)
- net GND: now also U13.3 (I0), C43.2, C45.2, C6.2, U10.2 (GND)
- net HEN: now also U14.3 (Y); no longer U12.4 (Z)
- net HF PWM: now also U17.7, TP2.1; no longer U17.6
- net Vtri: now also U17.2 (-); no longer U17.4 (-)
- net at C5.1, R10.2, R11.1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: now also U17.1 (+); no longer U17.3 (+)
- new net: U10.1 (I1), U9.4 (Z)
- new net: U12.4 (Z), U14.1 (A)
- new net: U13.4 (Z), U14.5 (B)
- new net Current_Dir: U10.3 (I0)
Other:
- note added: "For 5x MUXES"
- note added: "For HIP"
- note removed: "2x 2:1 EN*C"
- moved on the sheet: C8, R15, U9

Commit message: PCB Almost done with one coil!!
Parts:
- removed C8: 2.2u, Capacitor_SMD:C_0603_1608Metric, symbol Device:C
- added C50: 100n, Capacitor_SMD:C_0603_1608Metric, symbol Device:C
Connections:
- net +5V: now also C50.1
- net GND: now also C50.2
Other:
- note added: "For 6x MUXES"
- note removed: "For 5x MUXES"
- moved on the sheet: C10, C43, C45, C6, C9

Commit message: HF PWM done for both coils
Other:
- note added: "- Internal connections done - Spacing, shorts, nets, etc verified - Grouped"
Changed lines of the file:
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@@
+		)
+	)
+	(text "- Internal connections done\n- Spacing, shorts, nets, etc verified\n- Grouped"
+		(exclude_from_sim no)
+		(at 39.116 127.508 0)
+		(effects
+			(font
+				(size 1.27 1.27)
+				(italic yes)
+				(color 0 194 0 1)
+			)
+			(justify left)
 		)
 	)
