File: KiCadV2/KiCadV2.kicad_pcb (KiCad board)
At the start: 2 copper layers, 151 parts, among them J1 USB_C_Receptacle_PowerOnly_6P, J2 Screw_Terminal_01x02, J3 Screw_Terminal_01x02, U1 MT3608, U19 HIP4080A, U2 74HC595, U20 DMHT10H032LFJ, U21 INA240A1D, U22 DMHT10H032LFJ, U23 INA240A1D, U31 HIP4080A, U32 MCP6002-xSN, U33 CJ432

Commit message: idk
Parts:
- removed C35, C36, C37, C40, C42: 100n, Capacitor_SMD:C_0603_1608Metric
- removed C38, C39: 1uF, Capacitor_SMD:C_0603_1608Metric
- removed C41, C43: 2.2u, Capacitor_SMD:C_0603_1608Metric
- removed D13: D, Diode_SMD:D_SMA
- removed R50, R51: 10k, Resistor_SMD:R_0603_1608Metric
- removed R52: 9200, Resistor_SMD:R_0603_1608Metric
- removed R53: 800, Resistor_SMD:R_0603_1608Metric
- removed R54, R55: 100, Resistor_SMD:R_0603_1608Metric
- removed U10: ~, Package_TO_SOT_SMD:SOT-363_SC-70-6
- removed U31: HIP4080A, Package_SO:SOIC-20W_7.5x12.8mm_P1.27mm
- removed U32: MCP6002-xSN, Package_SO:SOIC-8_3.9x4.9mm_P1.27mm
- removed U33: CJ432, Package_TO_SOT_SMD:SOT-23
- added J4: Screw_Terminal_01x02, Connector_PinHeader_2.54mm:PinHeader_2x01_P2.54mm_Vertical, F.Cu at (111.8, 98.3)
- C10, C26: value 100n -> 470p
- C16, C17: value 1uF -> 100n
- C19, C23, C29, C30, C7: value 2.2u -> 100n
- C22, C6: value 100n -> 33n
- C24, C25, C33, C34: value 100n -> 2.2u
- C27, C5: value C -> 100n
- C31: value 470p -> 100n
- C9: value 470p -> 2.2u
- D2: value D -> D_Schottky
- D4: value LED -> D; footprint LED_SMD:LED_0603_1608Metric -> Diode_SMD:D_SMA
- D5: value LED -> KT-0603W
- D6: value D -> KT-0603W; footprint Diode_SMD:D_SMA -> LED_SMD:LED_0603_1608Metric
- R10, R9: value 12.25k -> 12k
- R11, R12, R49: value 250 -> 100
- R13, R14: value 400 -> 390
- R15: value R -> 2700
- R16: value R -> 1500
- R17: value R -> 2000
- R2: value 19k -> 18k
- R22: value 10k -> 51k
- R23: value 50k -> 51k
- R24: value 50k -> 0.1; footprint Resistor_SMD:R_0603_1608Metric -> Resistor_SMD:R_1206_3216Metric
- R25: value 2k -> 0.1; footprint Resistor_SMD:R_0603_1608Metric -> Resistor_SMD:R_1206_3216Metric
- R26: value 2k -> 820
- R27, R28: value 0.1 -> 1k; footprint Resistor_SMD:R_1206_3216Metric -> Resistor_SMD:R_0603_1608Metric
- R29: value 820 -> 0.1; footprint Resistor_SMD:R_0603_1608Metric -> Resistor_SMD:R_1206_3216Metric
- R30: value 1k -> 0.1; footprint Resistor_SMD:R_0603_1608Metric -> Resistor_SMD:R_1206_3216Metric
- R31: value 1k -> 820
- R32, R33: value 2k -> 1k
- R34: value 0.1 -> 2700; footprint Resistor_SMD:R_1206_3216Metric -> Resistor_SMD:R_0603_1608Metric
- R35: value 0.1 -> 1500; footprint Resistor_SMD:R_1206_3216Metric -> Resistor_SMD:R_0603_1608Metric
- R36: value 820 -> 2000
- R38: value 1k -> 9.1k
- R39: value R -> 5.1k
- R40: value R -> 10k
- R41: value R -> 51k
- R42: value 1k -> 51k
- R43: value 9.1k -> 200; footprint Resistor_SMD:R_0603_1608Metric -> Resistor_SMD:R_0805_2012Metric
- R44: value 5.1k -> 10k
- R46: value 10k -> 9.1k
- R47: value 50k -> 820
- R48: value 50k -> 100
- U11: value ~ -> MX3502S; footprint Package_TO_SOT_SMD:SOT-363_SC-70-6 -> Package_SO:SOP-8_3.76x4.96mm_P1.27mm
- U12, U24: value ~ -> NC7SZ157P6X; footprint Package_SO:SOP-8_3.76x4.96mm_P1.27mm -> Package_TO_SOT_SMD:SOT-363_SC-70-6
- U13, U14, U15, U16, U25, U26, U27, U3, U4, U5: value ~ -> NC7SZ157P6X
- U17, U28: value ~ -> HIP4080A; footprint Package_TO_SOT_SMD:SOT-363_SC-70-6 -> Package_SO:SOIC-20W_7.5x12.8mm_P1.27mm
- U18: value ~ -> DMHT10H032LFJ; footprint Package_TO_SOT_SMD:SOT-363_SC-70-6 -> Module:V-DFN5045-12
- U19: value HIP4080A -> INA240A1D; footprint Package_SO:SOIC-20W_7.5x12.8mm_P1.27mm -> Package_SO:SOIC-8_3.9x4.9mm_P1.27mm
- U22: value DMHT10H032LFJ -> MX3502S; footprint Module:V-DFN5045-12 -> Package_SO:SOP-8_3.76x4.96mm_P1.27mm
- U23: value INA240A1D -> NC7SZ157P6X; footprint Package_SO:SOIC-8_3.9x4.9mm_P1.27mm -> Package_TO_SOT_SMD:SOT-363_SC-70-6
- U29: value ~ -> MCP6002-xSN; footprint Package_TO_SOT_SMD:SOT-363_SC-70-6 -> Package_SO:SOIC-8_3.9x4.9mm_P1.27mm
- U30: value ~ -> CJ432; footprint Package_TO_SOT_SMD:SOT-363_SC-70-6 -> Package_TO_SOT_SMD:SOT-23
- U6: value ~ -> 74LV08AT14-13; footprint Package_TO_SOT_SMD:SOT-363_SC-70-6 -> Package_SO:TSSOP-14_4.4x5mm_P0.65mm
- U7: value ~ -> DAC082S085CISDX/NOPB; footprint Package_TO_SOT_SMD:SOT-363_SC-70-6 -> Package_SON:WSON-10-1EP_3x3mm_P0.5mm_EP1.6x2mm
- U8: value ~ -> MX3502S; footprint Package_SON:WSON-10-1EP_3x3mm_P0.5mm_EP1.6x2mm -> Package_SO:SOP-8_3.76x4.96mm_P1.27mm
- U9: value ~ -> GT74LVC6G14TD; footprint Package_SO:SOP-8_3.76x4.96mm_P1.27mm -> Package_SO:TSSOP-14_4.4x5mm_P0.65mm
- moved D4 171.7 mm to (79.3, 102.7)
- moved D1 141.8 mm to (79.3, 89.1)
- moved D2 141.8 mm to (79.3, 93.6)
- moved D3 141.8 mm to (79.3, 98.2)
- moved C21 134.0 mm to (112.6, 108.2)
- moved U12 129.6 mm to (77.3, 109.0)
- moved U24 129.1 mm to (108.5, 112.9)
- moved J2 124.2 mm to (111.8, 89.1)
- moved J3 124.2 mm to (111.8, 93.7)
- moved U9 123.7 mm to (121.0, 96.9)
- moved U1 123.4 mm to (132.2, 100.8)
- moved C10 110.9 mm to (81.4, 120.8)
- moved C11 110.9 mm to (81.4, 123.3)
- moved C16 110.8 mm to (85.5, 118.3)
- moved R19 110.8 mm to (89.5, 113.3)
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Connections:
- C10 pad 1: +5V -> /PerCoil/SignalProcessingChain/Vtri
- C13 pad 1: +5V -> +12V
- C14 pad 1: +5V -> /VCM
- C15 pad 1: +12V -> Net-(D7-K)
- C15 pad 2: GND -> /+OUT1
- C16 pad 1: Net-(D7-K) -> Net-(D8-K)
- C16 pad 2: /+OUT1 -> /PerCoil/BHS
- C17 pad 1: Net-(D8-K) -> GND
- C17 pad 2: /PerCoil/BHS -> /A1
- C18 pad 1: GND -> Net-(U19--)
- C18 pad 2: /PerCoil/SignalProcessingChain/VCM -> Net-(U19-+)
- C19 pad 2: /PerCoil/SignalProcessingChain/VCM -> /A2
- C20 pad 1: GND -> Net-(U21--)
- C20 pad 2: /A1 -> Net-(U21-+)
- C21 pad 1: Net-(U21--) -> /VCM
- C21 pad 2: Net-(U21-+) -> GND
- C22 pad 1: GND -> Net-(U22B-+)
- C22 pad 2: /PerCoil1/SignalProcessingChain/VCM -> GND
- C23 pad 1: GND -> +5V
- C23 pad 2: /PerCoil1/SignalProcessingChain/VCM -> GND
- C24 pad 1: GND -> +5V
- C24 pad 2: /A2 -> GND
- C25 pad 1: Net-(U23--) -> +5V
- C25 pad 2: Net-(U23-+) -> GND
- C26 pad 1: /PerCoil1/SignalProcessingChain/VCM -> /PerCoil1/SignalProcessingChain/Vtri
- C27 pad 1: Net-(U24B-+) -> +5V
- C29 pad 1: +5V -> +12V
- C30 pad 1: +5V -> /VCM
- C31 pad 1: Net-(U24A--) -> Net-(D11-K)
- C31 pad 2: GND -> /+OUT2
- C32 pad 1: +5V -> Net-(D12-K)
- C32 pad 2: GND -> /PerCoil1/BHS
- C33 pad 1: +5V -> GND
- C33 pad 2: GND -> /VCM
- C34 pad 1: +5V -> GND
- C34 pad 2: GND -> /0.2V
- C4 pad 1: /PerCoil/SignalProcessingChain/VCM -> GND
- C4 pad 2: GND -> /0.2V
- C5 pad 1: Net-(U12B-+) -> /VCM
- C6 pad 1: +5V -> Net-(U11B-+)
- C9 pad 1: Net-(U12A--) -> +5V
- D11 pad 1: /PerCoil1/EN -> Net-(D11-K)
- D11 pad 2: /PerCoil1/SignalProcessingChain/EN*C -> +12V
- D2 pad 1: Net-(D2-K) -> VBUS
- D2 pad 2: /B1 -> GND
- D3 pad 1: Net-(D2-K) -> Net-(D3-K)
- D3 pad 2: /C1 -> /B1
- D4 pad 1: GND -> Net-(D3-K)
- D4 pad 2: Net-(D4-A) -> /C1
- D6 pad 1: /PerCoil/EN -> GND
- D6 pad 2: /PerCoil/SignalProcessingChain/EN*C -> Net-(D6-A)
- J2 pad 1: /+OUT1 -> VBUS
- J2 pad 2: /-OUT1 -> GND
- J3 pad 1: /+OUT2 -> /+OUT1
- J3 pad 2: /-OUT2 -> /-OUT1
- L2 pad 2: Net-(U21--) -> Net-(U19--)
- L3 pad 2: Net-(U23--) -> Net-(U21--)
- R10 pad 1: Net-(U9B-+) -> Net-(U8B-+)
- R11 pad 2: Net-(U9A-+) -> Net-(U8A-+)
- R12 pad 2: Net-(U9B-+) -> Net-(U8B-+)
- R13 pad 1: Net-(D4-A) -> Net-(D5-A)
- R13 pad 2: Net-(U10-Z) -> Net-(R13-Pad2)
- R14 pad 1: Net-(D5-A) -> Net-(D6-A)
- R14 pad 2: Net-(U11-Z) -> Net-(R14-Pad2)
- R15 pad 2: Net-(U12B-+) -> Net-(U11B-+)
- R16 pad 1: Net-(U12B-+) -> Net-(U11B-+)
- R17 pad 2: Net-(U12B-+) -> Net-(U11B-+)
- R18 pad 1: /PerCoil/SignalProcessingChain/VCM -> /VCM
- R18 pad 2: /PerCoil/SignalProcessingChain/Vtri -> Net-(U11A-+)
- R19 pad 1: /PerCoil/SignalProcessingChain/Vtri -> Net-(U11A-+)
- R20 pad 1: Net-(U12A--) -> /PerCoil/SignalProcessingChain/Vtri
- R21 pad 1: /C1 -> VBUS
- R21 pad 2: /PerCoil/SignalProcessingChain/EN*C -> /PerCoil/SignalProcessingChain/DIS
- R22 pad 1: VBUS -> Net-(U17-HDEL)
- R22 pad 2: /PerCoil/SignalProcessingChain/DIS -> GND
- R23 pad 1: Net-(U19-HDEL) -> Net-(U17-LDEL)
- R24 pad 1: Net-(U19-LDEL) -> /PerCoil/OC_SENSE
- R25 pad 1: +5V -> Net-(U19--)
- R25 pad 2: /PerCoil/SignalProcessingChain/VCM -> /-OUT1
- R26 pad 1: /PerCoil/SignalProcessingChain/VCM -> Net-(U19--)
- R26 pad 2: GND -> Net-(U19-+)
- R27 pad 1: /PerCoil/OC_SENSE -> /A1
- R27 pad 2: GND -> Net-(R27-Pad2)
- R28 pad 1: Net-(U21--) -> /-OUT1
- R28 pad 2: /-OUT1 -> Net-(U19-+)
- R29 pad 1: Net-(U21--) -> /PerCoil1/OC_SENSE
- R29 pad 2: Net-(U21-+) -> GND
- R30 pad 1: /A1 -> Net-(U21--)
- R30 pad 2: Net-(R30-Pad2) -> /-OUT2
- R31 pad 1: /-OUT1 -> Net-(U21--)
- R32 pad 1: +5V -> /A2
- R32 pad 2: /PerCoil1/SignalProcessingChain/VCM -> Net-(R32-Pad2)
- R33 pad 1: /PerCoil1/SignalProcessingChain/VCM -> /-OUT2
- R33 pad 2: GND -> Net-(U21-+)
- R34 pad 1: /PerCoil1/OC_SENSE -> /DACOUT2
- R34 pad 2: GND -> Net-(U22B-+)
- R35 pad 1: Net-(U23--) -> Net-(U22B-+)
- R35 pad 2: /-OUT2 -> +5V
- R36 pad 1: Net-(U23--) -> GND
- R36 pad 2: Net-(U23-+) -> Net-(U22B-+)
- R37 pad 1: /A2 -> /VCM
- R37 pad 2: Net-(R37-Pad2) -> Net-(U22A-+)
- R38 pad 1: /-OUT2 -> Net-(U22A-+)
- R38 pad 2: Net-(U23-+) -> /PerCoil1/SignalProcessingChain/Vsq
- R39 pad 1: /DACOUT2 -> /PerCoil1/SignalProcessingChain/Vtri
- R39 pad 2: Net-(U24B-+) -> /PerCoil1/SignalProcessingChain/Vsq
- R40 pad 1: Net-(U24B-+) -> VBUS
- R40 pad 2: +5V -> /PerCoil1/SignalProcessingChain/DIS
- R41 pad 1: GND -> Net-(U28-HDEL)
- R41 pad 2: Net-(U24B-+) -> GND
- R42 pad 1: /PerCoil1/SignalProcessingChain/VCM -> Net-(U28-LDEL)
- R42 pad 2: /PerCoil1/SignalProcessingChain/Vtri -> GND
- R43 pad 1: /PerCoil1/SignalProcessingChain/Vtri -> +5V
- R43 pad 2: /PerCoil1/SignalProcessingChain/Vsq -> Net-(U30-K)
- R44 pad 1: Net-(U24A--) -> +5V
- R44 pad 2: /PerCoil1/SignalProcessingChain/Vsq -> Net-(U29A-+)
- R45 pad 1: /C2 -> Net-(U29A-+)
- R45 pad 2: /PerCoil1/SignalProcessingChain/EN*C -> GND
- R46 pad 1: VBUS -> Net-(U30-K)
- R46 pad 2: /PerCoil1/SignalProcessingChain/DIS -> Net-(U29B-+)
- R47 pad 1: Net-(U31-HDEL) -> Net-(U29B-+)
- R48 pad 1: Net-(U31-LDEL) -> Net-(U29A--)
- R48 pad 2: GND -> /VCM
- R49 pad 1: +5V -> Net-(U29B--)
- R49 pad 2: Net-(U33-K) -> /0.2V
- R6 pad 1: /EN1 -> Net-(D3-K)
- R7 pad 1: /EN2 -> /EN1
- R8 pad 1: Net-(D2-K) -> /EN2
- R9 pad 1: Net-(U9A-+) -> Net-(U8A-+)
- U11 pad 1: GND -> Net-(U11A-+)
- U11 pad 2: GND -> /PerCoil/SignalProcessingChain/Vtri
- U11 pad 3: +5V -> Net-(U11B-+)
- U11 pad 4: Net-(U11-Z) -> /PerCoil/SignalProcessingChain/Vtri
- U11 pad 5: +5V -> GND
- U11 pad 6: /~{OC2} -> /PerCoil/SignalProcessingChain/HF PWM
- U12 pad 1: /PerCoil/SignalProcessingChain/Vtri -> /PerCoil/SignalProcessingChain/HF PWM
- U12 pad 2: Net-(U12A--) -> GND
- U12 pad 3: Net-(U12B-+) -> /PWM2
- U12 pad 4: /PerCoil/SignalProcessingChain/Vtri -> Net-(U12-Z)
- U12 pad 5: GND -> +5V
- U12 pad 6: /PerCoil/SignalProcessingChain/HF PWM -> /B1
- U13 pad 3: /PWM2 -> /PWM1
- U13 pad 4: Net-(U13-Z) -> /PerCoil/SignalProcessingChain/DIR
- U13 pad 6: /B1 -> /A1
- U14 pad 1: /PerCoil/SignalProcessingChain/HF PWM -> /PWM2
- U14 pad 3: /PWM1 -> Net-(U12-Z)
- U14 pad 4: /PerCoil/SignalProcessingChain/DIR -> Net-(U14-Z)
- U15 pad 1: /PWM2 -> +5V
- U15 pad 3: Net-(U13-Z) -> Net-(U14-Z)
- U15 pad 4: Net-(U15-Z) -> /PerCoil/SignalProcessingChain/HEN
- U15 pad 6: /A1 -> /C1
- U16 pad 1: GND -> Net-(U14-Z)
- U16 pad 3: +5V -> Net-(U16-I0)
- U16 pad 4: Net-(U16-Z) -> /PerCoil/SignalProcessingChain/DIS
- U16 pad 6: /PerCoil/EN -> /PerCoil/SignalProcessingChain/EN*C
- U17 pad 1: +5V -> Net-(D8-K)
- U17 pad 2: GND -> /PerCoil/SignalProcessingChain/HEN
- U17 pad 3: Net-(U15-Z) -> /PerCoil/SignalProcessingChain/DIS
- U17 pad 4: /PerCoil/SignalProcessingChain/HEN -> GND
- U17 pad 5: +5V -> /PerCoil/SignalProcessingChain/Out
- U17 pad 6: /C1 -> /PerCoil/SignalProcessingChain/DIR
- U18 pad 1: Net-(U15-Z) -> /PerCoil/AH
- U18 pad 2: GND -> VBUS
- U18 pad 3: Net-(U16-Z) -> /+OUT1
- U18 pad 4: /PerCoil/SignalProcessingChain/DIS -> /PerCoil/AL
- U18 pad 5: +5V -> /PerCoil/OC_SENSE
- U18 pad 6: /PerCoil/SignalProcessingChain/EN*C -> /PerCoil/OC_SENSE
- U19 pad 1: Net-(D8-K) -> Net-(U19--)
- U19 pad 2: /PerCoil/SignalProcessingChain/HEN -> GND
- U19 pad 3: /PerCoil/SignalProcessingChain/DIS -> GND
- U19 pad 5: /PerCoil/SignalProcessingChain/Out -> Net-(R27-Pad2)
- U19 pad 6: /PerCoil/SignalProcessingChain/DIR -> +5V
- U19 pad 7: /VCM -> +5V
- U19 pad 8: Net-(U19-HDEL) -> Net-(U19-+)
- U20 pad 1: /PerCoil/AH -> /PerCoil1/AH
- U20 pad 10: /PerCoil/BH -> /PerCoil1/BH
- U20 pad 3: /+OUT1 -> /+OUT2
- U20 pad 4: /PerCoil/AL -> /PerCoil1/AL
- U20 pad 5: /PerCoil/OC_SENSE -> /PerCoil1/OC_SENSE
- U20 pad 6: /PerCoil/OC_SENSE -> /PerCoil1/OC_SENSE
- U20 pad 7: /PerCoil/BL -> /PerCoil1/BL
- U20 pad 8: /PerCoil/BHS -> /PerCoil1/BHS
- U21 pad 5: Net-(R30-Pad2) -> Net-(R32-Pad2)
- U22 pad 1: /PerCoil1/AH -> Net-(U22A-+)
- U22 pad 2: VBUS -> /PerCoil1/SignalProcessingChain/Vtri
- U22 pad 3: /+OUT2 -> Net-(U22B-+)
- U22 pad 4: /PerCoil1/AL -> /PerCoil1/SignalProcessingChain/Vtri
- U22 pad 5: /PerCoil1/OC_SENSE -> GND
- U22 pad 6: /PerCoil1/OC_SENSE -> /PerCoil1/SignalProcessingChain/HF PWM
- U22 pad 7: /PerCoil1/BL -> /PerCoil1/SignalProcessingChain/Vsq
- U22 pad 8: /PerCoil1/BHS -> +5V
- U23 pad 1: Net-(U23--) -> /PerCoil1/SignalProcessingChain/HF PWM
- U23 pad 3: GND -> /PWM4
- U23 pad 4: GND -> Net-(U23-Z)
- U23 pad 5: Net-(R37-Pad2) -> +5V
- U23 pad 6: +5V -> /B2
- U24 pad 1: /PerCoil1/SignalProcessingChain/Vtri -> /PerCoil1/SignalProcessingChain/HF PWM
- U24 pad 2: Net-(U24A--) -> GND
- U24 pad 3: Net-(U24B-+) -> /PWM3
- U24 pad 4: /PerCoil1/SignalProcessingChain/Vtri -> /PerCoil1/SignalProcessingChain/DIR
- U24 pad 5: GND -> +5V
- U24 pad 6: /PerCoil1/SignalProcessingChain/HF PWM -> /A2
- U25 pad 1: /PerCoil1/SignalProcessingChain/HF PWM -> /PWM4
- U25 pad 3: /PWM4 -> Net-(U23-Z)
- U25 pad 6: /B2 -> /A2
- U26 pad 1: /PerCoil1/SignalProcessingChain/HF PWM -> +5V
- U26 pad 3: /PWM3 -> Net-(U25-Z)
- U26 pad 4: /PerCoil1/SignalProcessingChain/DIR -> /PerCoil1/SignalProcessingChain/HEN
- U26 pad 6: /A2 -> /C2
- U27 pad 1: /PWM4 -> Net-(U25-Z)
- U27 pad 3: Net-(U25-Z) -> Net-(U27-I0)
- U27 pad 4: Net-(U27-Z) -> /PerCoil1/SignalProcessingChain/DIS
- U27 pad 6: /A2 -> /PerCoil1/SignalProcessingChain/EN*C
- U28 pad 1: GND -> Net-(D12-K)
- U28 pad 2: GND -> /PerCoil1/SignalProcessingChain/HEN
- U28 pad 3: +5V -> /PerCoil1/SignalProcessingChain/DIS
- U28 pad 4: Net-(U28-Z) -> GND
- U28 pad 5: +5V -> /PerCoil1/SignalProcessingChain/Out
- U28 pad 6: /PerCoil1/EN -> /PerCoil1/SignalProcessingChain/DIR
- U29 pad 1: +5V -> Net-(U29A--)
- U29 pad 2: GND -> Net-(U29A--)
- U29 pad 3: Net-(U27-Z) -> Net-(U29A-+)
- U29 pad 4: /PerCoil1/SignalProcessingChain/HEN -> GND
- U29 pad 5: +5V -> Net-(U29B-+)
- U29 pad 6: /C2 -> Net-(U29B--)
- U30 pad 1: Net-(U27-Z) -> Net-(U30-K)
- U30 pad 2: GND -> Net-(U30-K)
- U30 pad 3: Net-(U28-Z) -> GND
- U5 pad 6: Net-(D2-K) -> Net-(D3-K)
- U6 pad 1: /~{OC1} -> /EN1
- U6 pad 2: GND -> /~{OC1}
- U6 pad 3: GND -> /PerCoil/EN
- U6 pad 4: /PerCoil/EN -> /EN2
- U6 pad 5: +5V -> /~{OC2}
- U6 pad 6: /EN1 -> /PerCoil1/EN
- U7 pad 1: /~{OC2} -> +5V
- U7 pad 2: GND -> /DACOUT1
- U7 pad 3: GND -> /DACOUT2
- U7 pad 4: /PerCoil1/EN -> unconnected-(U7-NC-Pad4)
- U7 pad 5: +5V -> unconnected-(U7-NC-Pad5)
- U7 pad 6: /EN2 -> GND
- U8 pad 1: +5V -> Net-(U8A-+)
- U8 pad 2: /DACOUT1 -> /PerCoil/OC_SENSE
- U8 pad 3: /DACOUT2 -> Net-(U8B-+)
- U8 pad 4: unconnected-(U8-NC-Pad4) -> /PerCoil1/OC_SENSE
- U8 pad 5: unconnected-(U8-NC-Pad5) -> GND
- U8 pad 6: GND -> /~{OC2}
- U8 pad 7: /VCM -> /~{OC1}
- U8 pad 8: Net-(U5-Z) -> +5V
- U9 pad 1: Net-(U9A-+) -> /~{OC1}
- U9 pad 2: /PerCoil/OC_SENSE -> Net-(R13-Pad2)
- U9 pad 3: Net-(U9B-+) -> /~{OC2}
- U9 pad 4: /PerCoil1/OC_SENSE -> Net-(R14-Pad2)
- U9 pad 5: GND -> /PerCoil/EN
- U9 pad 6: /~{OC2} -> Net-(U16-I0)
- U9 pad 7: /~{OC1} -> unconnected-(U9G-GND-Pad7)
- U9 pad 8: +5V -> Net-(U27-I0)

Commit message: PCB Almost done with one coil!!
Parts:
- removed C22: 33n, Capacitor_SMD:C_0603_1608Metric
- removed C8: 2.2u, Capacitor_SMD:C_0603_1608Metric
- removed R47: 820, Resistor_SMD:R_0603_1608Metric
- removed R48, R49: 100, Resistor_SMD:R_0603_1608Metric
- removed U16, U24, U25, U27: NC7SZ157P6X, Package_TO_SOT_SMD:SOT-363_SC-70-6
- removed U19: INA240A1D, Package_SO:SOIC-8_3.9x4.9mm_P1.27mm
- added C35: 100n, Capacitor_SMD:C_0603_1608Metric, F.Cu at (23.6, 116.7)
- added C36: 100n, Capacitor_SMD:C_0603_1608Metric, F.Cu at (23.6, 119.2)
- added C37: 2.2u, Capacitor_SMD:C_0603_1608Metric, F.Cu at (23.6, 121.7)
- added C38: 2.2u, Capacitor_SMD:C_0603_1608Metric, F.Cu at (23.6, 124.2)
- added C39: 100n, Capacitor_SMD:C_0603_1608Metric, F.Cu at (151.4, 18.2)
- added C40: 100n, Capacitor_SMD:C_0603_1608Metric, F.Cu at (157.2, 24.0)
- added C41: 100n, Capacitor_SMD:C_0603_1608Metric, F.Cu at (157.2, 26.5)
- added C42: 2.2u, Capacitor_SMD:C_0603_1608Metric, F.Cu at (157.2, 29.0)
- added C43: 100n, Capacitor_SMD:C_0603_1608Metric, F.Cu at (84.4, 181.3)
- added C44: 100n, Capacitor_SMD:C_0603_1608Metric, F.Cu at (133.4, 104.7)
- added C45: 100n, Capacitor_SMD:C_0603_1608Metric, F.Cu at (76.4, 181.3)
- added C46: 100n, Capacitor_SMD:C_0603_1608Metric, F.Cu at (133.4, 107.2)
- added C47: 100n, Capacitor_SMD:C_0603_1608Metric, F.Cu at (64.4, 170.3)
- added C48: 100n, Capacitor_SMD:C_0603_1608Metric, F.Cu at (188.5, 105.9)
- added C49: 100n, Capacitor_SMD:C_0603_1608Metric, F.Cu at (159.5, 116.0)
- added C50: 100n, Capacitor_SMD:C_0603_1608Metric, F.Cu at (82.5, 177.8)
- added C51: 100n, Capacitor_SMD:C_0603_1608Metric, F.Cu at (133.4, 109.7)
- added D13: D_bootstrap, Diode_SMD:D_SOD-523, F.Cu at (141.2, 106.6)
- added TP1: TestPoint, TestPoint:TestPoint_Pad_D2.5mm, F.Cu at (151.0, 25.8)
- added TP2: TestPoint, TestPoint:TestPoint_Pad_D2.5mm, B.Cu at (126.9, 182.6)
- added TP3: TestPoint, TestPoint:TestPoint_Pad_D2.5mm, F.Cu at (141.7, 100.7)
- added U10: NC7SZ157P6X, Package_TO_SOT_SMD:SOT-363_SC-70-6, F.Cu at (85.0, 172.4)
- added U31: INA240A1D, Package_SO:SOIC-8_3.9x4.9mm_P1.27mm, F.Cu at (178.0, 103.6)
- added U32: NC7SZ157P6X, Package_TO_SOT_SMD:SOT-363_SC-70-6, F.Cu at (125.3, 85.9)
- added U33: NC7SZ157P6X, Package_TO_SOT_SMD:SOT-363_SC-70-6, F.Cu at (125.3, 89.9)
- added U34: NC7SZ157P6X, Package_TO_SOT_SMD:SOT-363_SC-70-6, F.Cu at (125.3, 93.8)
- added U35: NC7SZ157P6X, Package_TO_SOT_SMD:SOT-363_SC-70-6, F.Cu at (125.3, 97.7)
- added U36: NC7SZ157P6X, Package_TO_SOT_SMD:SOT-363_SC-70-6, F.Cu at (125.3, 101.6)
- added U37: NC7SZ157P6X, Package_TO_SOT_SMD:SOT-363_SC-70-6, F.Cu at (125.3, 105.6)
- added U38: 74LV08AT14-13, Package_SO:TSSOP-14_4.4x5mm_P0.65mm, F.Cu at (162.2, 101.2)
- added U39: HIP4080A, Package_SO:SOIC-20W_7.5x12.8mm_P1.27mm, F.Cu at (133.9, 91.2)
- added U40: MCP6002-xSN, Package_SO:SOIC-8_3.9x4.9mm_P1.27mm, F.Cu at (25.1, 80.4)
- added U41: CJ432, Package_TO_SOT_SMD:SOT-23, F.Cu at (23.3, 85.8)
- A1: footprint Module:Arduino_UNO_R3 -> Module:Arduino_UNO_R3_ConnOnly
- C1: value 22uF -> 100uF
- C10, C26: value 470p -> 100n
- C19, C5: value 100n -> 33n
- C2: value 100n -> 22uF; footprint Capacitor_SMD:C_0603_1608Metric -> Capacitor_SMD:C_1206_3216Metric
- C20, C21, C29: value 100n -> 2.2u
- C24, C25, C3, C33, C34, C9: value 2.2u -> 100n
- C4: value 100n -> 470p
- C6: value 33n -> 100n
- D1: value D -> D_power; footprint Diode_SMD:D_SMA -> Diode_SMD:D_SOD-123
- D10: value D_Schottky -> KT-0603W; footprint Diode_SMD:D_SMA -> LED_SMD:LED_0603_1608Metric
- D11: value D -> D_Schottky; footprint Diode_SMD:D_SMA -> Diode_SMD:D_SOD-323
- D12, D7: value D -> D_bootstrap; footprint Diode_SMD:D_SMA -> Diode_SMD:D_SOD-523
- D2: value D_Schottky -> D_Power_Big; footprint Diode_SMD:D_SMA -> Diode_SMD:D_SMC
- D3: value D -> D_5.1V; footprint Diode_SMD:D_SMA -> Diode_SMD:D_SMB
- D4: value D -> D_logic
- D5: value KT-0603W -> D_logic; footprint LED_SMD:LED_0603_1608Metric -> Diode_SMD:D_SMA
- D6: value KT-0603W -> D_bootstrap; footprint LED_SMD:LED_0603_1608Metric -> Diode_SMD:D_SOD-523
- D8: value D -> KT-0603W; footprint Diode_SMD:D_SMA -> LED_SMD:LED_0603_1608Metric
- D9: footprint Diode_SMD:D_SMA -> Diode_SMD:D_SOD-323
- L1: value L -> 10u; footprint Inductor_THT:L_Axial_L5.3mm_D2.2mm_P2.54mm_Vertical_Vishay_IM-1 -> Inductor_SMD:10uH C15029
- L2, L3: footprint Inductor_SMD:L_TDK_SLF12555 -> Inductor_SMD:6.8uH C5127257
- R10: value 12k -> 2700
- R11: value 100 -> 1500
- R12: value 100 -> 2000
- R13, R14: value 390 -> 51k
- R15: value 2700 -> 10k
- R16: value 1500 -> 12k
- R17: value 2000 -> 10k
- R18, R27: value 1k -> 100
- R19: value 9.1k -> 390
- R2: value 18k -> 5.1k
- R20: value 5.1k -> 0.1; footprint Resistor_SMD:R_0603_1608Metric -> Resistor_SMD:R_1206_3216Metric
- R21: value 10k -> 0.1; footprint Resistor_SMD:R_0603_1608Metric -> Resistor_SMD:R_1206_3216Metric
- R22: value 51k -> 820
- R23: value 51k -> 1k
- R24: value 0.1 -> 1k; footprint Resistor_SMD:R_1206_3216Metric -> Resistor_SMD:R_0603_1608Metric
- R25: value 0.1 -> 12k; footprint Resistor_SMD:R_1206_3216Metric -> Resistor_SMD:R_0603_1608Metric
- R26: value 820 -> 10k
- R28: value 1k -> 390
- R3: value 1k -> 18k
- R37: value 1k -> 51k
- R38: value 9.1k -> 51k
- R39: value 5.1k -> 10k
- R4: value 5.1k -> 1k
- R40: value 10k -> 200; footprint Resistor_SMD:R_0603_1608Metric -> Resistor_SMD:R_0805_2012Metric
- R41, R42: value 51k -> 10k
- R43: value 200 -> 9.1k; footprint Resistor_SMD:R_0805_2012Metric -> Resistor_SMD:R_0603_1608Metric
- R44: value 10k -> 820
- R45: value 10k -> 100
- R46: value 9.1k -> 100
- R6: value 10k -> 1k
- R7: value 10k -> 9.1k
- R8: value 10k -> 5.1k
- R9: value 12k -> 10k
- U11, U8: value MX3502S -> NC7SZ157P6X; footprint Package_SO:SOP-8_3.76x4.96mm_P1.27mm -> Package_TO_SOT_SMD:SOT-363_SC-70-6
- U14: value NC7SZ157P6X -> 74LV08AT14-13; footprint Package_TO_SOT_SMD:SOT-363_SC-70-6 -> Package_SO:TSSOP-14_4.4x5mm_P0.65mm
- U15: value NC7SZ157P6X -> HIP4080A; footprint Package_TO_SOT_SMD:SOT-363_SC-70-6 -> Package_SO:SOIC-20W_7.5x12.8mm_P1.27mm
- U17: value HIP4080A -> MX3502S; footprint Package_SO:SOIC-20W_7.5x12.8mm_P1.27mm -> Package_SO:SOP-8_3.76x4.96mm_P1.27mm
- U18: value DMHT10H032LFJ -> MX3502S; footprint Module:V-DFN5045-12 -> Package_SO:SOP-8_3.76x4.96mm_P1.27mm
- U20: value DMHT10H032LFJ -> ~; footprint Module:V-DFN5045-12 -> TestPoint:SPDT_solder_bridge
- U21: value INA240A1D -> ~; footprint Package_SO:SOIC-8_3.9x4.9mm_P1.27mm -> TestPoint:SPDT_solder_bridge
- U22: value MX3502S -> DMHT10H032LFJ; footprint Package_SO:SOP-8_3.76x4.96mm_P1.27mm -> Module:V-DFN5045-12
- U23: value NC7SZ157P6X -> INA240A1D; footprint Package_TO_SOT_SMD:SOT-363_SC-70-6 -> Package_SO:SOIC-8_3.9x4.9mm_P1.27mm
- U26, U5: value NC7SZ157P6X -> MX3502S; footprint Package_TO_SOT_SMD:SOT-363_SC-70-6 -> Package_SO:SOP-8_3.76x4.96mm_P1.27mm
- U28: value HIP4080A -> ~; footprint Package_SO:SOIC-20W_7.5x12.8mm_P1.27mm -> TestPoint:SPDT_solder_bridge
- U29: value MCP6002-xSN -> ~; footprint Package_SO:SOIC-8_3.9x4.9mm_P1.27mm -> TestPoint:SPDT_solder_bridge
- U30: value CJ432 -> DMHT10H032LFJ; footprint Package_TO_SOT_SMD:SOT-23 -> Module:V-DFN5045-12
- U6: value 74LV08AT14-13 -> NC7SZ157P6X; footprint Package_SO:TSSOP-14_4.4x5mm_P0.65mm -> Package_TO_SOT_SMD:SOT-363_SC-70-6
- U9: value GT74LVC6G14TD -> NC7SZ157P6X; footprint Package_SO:TSSOP-14_4.4x5mm_P0.65mm -> Package_TO_SOT_SMD:SOT-363_SC-70-6
- moved R43 156.3 mm to (18.9, 85.8)
- moved C20 152.8 mm to (19.6, 119.2)
- moved R44 149.0 mm to (18.9, 88.3)
- moved R45 149.0 mm to (18.9, 90.8)
- moved R46 149.0 mm to (18.9, 93.3)
- moved J4 143.7 mm to (235.2, 24.6)
- moved J2 141.4 mm to (235.2, 20.0)
- moved C34 136.2 mm to (23.6, 114.2)
- moved A1 135.9 mm to (246.1, 39.0)
- moved R24 131.2 mm to (68.9, 161.9), turned to -90 degrees
- moved C1 130.2 mm to (40.8, 19.5)
- moved L1 125.5 mm to (24.1, 47.1)
- moved D4 121.0 mm to (171.0, 23.9)
- moved U21 116.2 mm to (59.3, 177.2), turned to 90 degrees
- moved U1 115.9 mm to (23.8, 59.6)
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Connections:
- C1 pad 1: +12V -> Vdrive
- C10 pad 1: /PerCoil/SignalProcessingChain/Vtri -> +5V
- C11 pad 1: +5V -> +12V
- C12 pad 1: +5V -> /VCM
- C13 pad 1: +12V -> Net-(D6-K)
- C13 pad 2: GND -> /+OUT1
- C14 pad 1: /VCM -> Net-(D7-K)
- C14 pad 2: GND -> /PerCoil/BHS
- C15 pad 1: Net-(D7-K) -> Net-(U23--)
- C15 pad 2: /+OUT1 -> Net-(U23-+)
- C16 pad 1: Net-(D8-K) -> GND
- C16 pad 2: /PerCoil/BHS -> /A1
- C17 pad 1: GND -> Net-(U31--)
- C17 pad 2: /A1 -> Net-(U31-+)
- C18 pad 1: Net-(U19--) -> GND
- C18 pad 2: Net-(U19-+) -> /A2
- C19 pad 1: GND -> Net-(U17B-+)
- C19 pad 2: /A2 -> GND
- C2 pad 1: GND -> +12V
- C2 pad 2: +5V -> GND
- C20 pad 1: Net-(U21--) -> +5V
- C20 pad 2: Net-(U21-+) -> GND
- C21 pad 1: /VCM -> +5V
- C25 pad 1: +5V -> +12V
- C26 pad 1: /PerCoil1/SignalProcessingChain/Vtri -> /VCM
- C27 pad 1: +5V -> Net-(D12-K)
- C27 pad 2: GND -> /+OUT2
- C28 pad 1: +5V -> Net-(D13-K)
- C28 pad 2: GND -> /PerCoil1/BHS
- C29 pad 1: +12V -> GND
- C29 pad 2: GND -> /VCM
- C3 pad 1: GND -> /VCM
- C3 pad 2: +5V -> GND
- C30 pad 1: /VCM -> GND
- C30 pad 2: GND -> /0.2V
- C31 pad 1: Net-(D11-K) -> +5V
- C31 pad 2: /+OUT2 -> GND
- C32 pad 1: Net-(D12-K) -> +5V
- C32 pad 2: /PerCoil1/BHS -> GND
- C33 pad 1: GND -> +5V
- C33 pad 2: /VCM -> GND
- C34 pad 1: GND -> +5V
- C34 pad 2: /0.2V -> GND
- C4 pad 1: GND -> /Vtri
- C4 pad 2: /0.2V -> GND
- C5 pad 1: /VCM -> Net-(U17A-+)
- C6 pad 1: Net-(U11B-+) -> +5V
- D10 pad 1: /PerCoil1/OC_SENSE -> Net-(D10-K)
- D10 pad 2: GND -> Net-(D10-A)
- D11 pad 1: Net-(D11-K) -> /PerCoil1/OC_SENSE
- D11 pad 2: +12V -> GND
- D2 pad 1: VBUS -> Vdrive
- D2 pad 2: GND -> Net-(D2-A)
- D3 pad 1: Net-(D3-K) -> Vdrive
- D3 pad 2: /B1 -> GND
- D4 pad 1: Net-(D3-K) -> Net-(D4-K)
- D4 pad 2: /C1 -> /B1
- D5 pad 1: GND -> Net-(D4-K)
- D5 pad 2: Net-(D5-A) -> /C1
- D6 pad 1: GND -> Net-(D6-K)
- D6 pad 2: Net-(D6-A) -> +12V
- D8 pad 2: +12V -> Net-(D8-A)
- J1 pad A9: VBUS -> Net-(D2-A)
- J1 pad B9: VBUS -> Net-(D2-A)
- L2 pad 2: Net-(U19--) -> Net-(U23--)
- L3 pad 2: Net-(U21--) -> Net-(U31--)
- R10 pad 1: Net-(U8B-+) -> /DACOUT1
- R10 pad 2: /~{OC2} -> Net-(U17A-+)
- R11 pad 1: /0.2V -> Net-(U17A-+)
- R11 pad 2: Net-(U8A-+) -> +5V
- R12 pad 1: /0.2V -> GND
- R12 pad 2: Net-(U8B-+) -> Net-(U17A-+)
- R13 pad 1: Net-(D5-A) -> Net-(U15-HDEL)
- R13 pad 2: Net-(R13-Pad2) -> GND
- R14 pad 1: Net-(D6-A) -> Net-(U15-LDEL)
- R14 pad 2: Net-(R14-Pad2) -> GND
- R15 pad 1: /DACOUT1 -> VBUS
- R15 pad 2: Net-(U11B-+) -> /PerCoil/SignalProcessingChain/DIS
- R16 pad 1: Net-(U11B-+) -> Net-(U18A-+)
- R16 pad 2: +5V -> /PerCoil/~{OC1}
- R17 pad 1: GND -> /EN1
- R17 pad 2: Net-(U11B-+) -> GND
- R18 pad 1: /VCM -> /0.2V
- R18 pad 2: Net-(U11A-+) -> Net-(U18A-+)
- R19 pad 1: Net-(U11A-+) -> Net-(D8-A)
- R19 pad 2: /PerCoil/SignalProcessingChain/Vsq -> +5V
- R2 pad 1: +12V -> Net-(J1-CC2)
- R2 pad 2: Net-(U1-FB) -> GND
- R20 pad 1: /PerCoil/SignalProcessingChain/Vtri -> /PerCoil/OC_SENSE
- R20 pad 2: /PerCoil/SignalProcessingChain/Vsq -> GND
- R21 pad 1: VBUS -> Net-(U23--)
- R21 pad 2: /PerCoil/SignalProcessingChain/DIS -> /-OUT1
- R22 pad 1: Net-(U17-HDEL) -> Net-(U23--)
- R22 pad 2: GND -> Net-(U23-+)
- R23 pad 1: Net-(U17-LDEL) -> /A1
- R23 pad 2: GND -> Net-(R23-Pad2)
- R24 pad 1: /PerCoil/OC_SENSE -> /-OUT1
- R24 pad 2: GND -> Net-(U23-+)
- R25 pad 1: Net-(U19--) -> Net-(U26B-+)
- R25 pad 2: /-OUT1 -> /PerCoil1/~{OC1}
- R26 pad 1: Net-(U19--) -> /EN2
- R26 pad 2: Net-(U19-+) -> GND
- R27 pad 1: /A1 -> /0.2V
- R27 pad 2: Net-(R27-Pad2) -> Net-(U26B-+)
- R28 pad 1: /-OUT1 -> Net-(D10-A)
- R28 pad 2: Net-(U19-+) -> +5V
- R3 pad 1: Net-(U1-FB) -> +12V
- R3 pad 2: GND -> Net-(U1-FB)
- R30 pad 1: Net-(U21--) -> Net-(U31--)
- R31 pad 1: Net-(U21--) -> Net-(U31--)
- R31 pad 2: Net-(U21-+) -> Net-(U31-+)
- R33 pad 2: Net-(U21-+) -> Net-(U31-+)
- R34 pad 2: Net-(U22B-+) -> Net-(U17B-+)
- R35 pad 1: Net-(U22B-+) -> Net-(U17B-+)
- R36 pad 2: Net-(U22B-+) -> Net-(U17B-+)
- R37 pad 1: /VCM -> Net-(U39-HDEL)
- R37 pad 2: Net-(U22A-+) -> GND
- R38 pad 1: Net-(U22A-+) -> Net-(U39-LDEL)
- R38 pad 2: /PerCoil1/SignalProcessingChain/Vsq -> GND
- R39 pad 1: /PerCoil1/SignalProcessingChain/Vtri -> VBUS
- R39 pad 2: /PerCoil1/SignalProcessingChain/Vsq -> /PerCoil1/SignalProcessingChain/DIS
- R4 pad 1: Net-(J1-CC1) -> Net-(U1-FB)
- R40 pad 1: VBUS -> +5V
- R40 pad 2: /PerCoil1/SignalProcessingChain/DIS -> Net-(U41-K)
- R41 pad 1: Net-(U28-HDEL) -> +5V
- R41 pad 2: GND -> Net-(U40A-+)
- R42 pad 1: Net-(U28-LDEL) -> Net-(U40A-+)
- R43 pad 1: +5V -> Net-(U41-K)
- R43 pad 2: Net-(U30-K) -> Net-(U40B-+)
- R44 pad 1: +5V -> Net-(U40B-+)
- R44 pad 2: Net-(U29A-+) -> GND
- R45 pad 1: Net-(U29A-+) -> Net-(U40A--)
- R45 pad 2: GND -> /VCM
- R46 pad 1: Net-(U30-K) -> Net-(U40B--)
- R46 pad 2: Net-(U29B-+) -> /0.2V
- R5 pad 1: Net-(J1-CC2) -> Net-(J1-CC1)
- R6 pad 1: Net-(D3-K) -> /VCM
- R6 pad 2: GND -> Net-(U5A-+)
- R7 pad 1: /EN1 -> Net-(U5A-+)
- R7 pad 2: GND -> /Vsq
- R8 pad 1: /EN2 -> /Vtri
- R8 pad 2: GND -> /Vsq
- R9 pad 1: Net-(U8A-+) -> Net-(D4-K)
- R9 pad 2: /~{OC1} -> GND
- U11 pad 1: Net-(U11A-+) -> /PWM2
- U11 pad 2: /PerCoil/SignalProcessingChain/Vtri -> GND
- U11 pad 3: Net-(U11B-+) -> Net-(U11-I0)
- U11 pad 4: /PerCoil/SignalProcessingChain/Vtri -> Net-(U11-Z)
- U11 pad 5: GND -> +5V
- U11 pad 6: /PerCoil/SignalProcessingChain/HF PWM -> /A1
- U12 pad 1: /PerCoil/SignalProcessingChain/HF PWM -> +5V
- U12 pad 3: /PWM2 -> Net-(U11-Z)
- U12 pad 6: /B1 -> /C1
- U13 pad 1: /PerCoil/SignalProcessingChain/HF PWM -> Net-(U11-Z)
- U13 pad 3: /PWM1 -> GND
- U13 pad 4: /PerCoil/SignalProcessingChain/DIR -> Net-(U13-Z)
- U13 pad 6: /A1 -> /C1
- U14 pad 1: /PWM2 -> Net-(U12-Z)
- U14 pad 2: GND -> /PerCoil/SignalProcessingChain/EN
- U14 pad 3: Net-(U12-Z) -> /PerCoil/SignalProcessingChain/HEN
- U14 pad 4: Net-(U14-Z) -> /PerCoil/SignalProcessingChain/EN
- U14 pad 5: +5V -> Net-(U13-Z)
- U14 pad 6: /A1 -> /PerCoil/SignalProcessingChain/DIS
- U15 pad 1: +5V -> Net-(D7-K)
- U15 pad 2: GND -> /PerCoil/SignalProcessingChain/HEN
- U15 pad 3: Net-(U14-Z) -> /PerCoil/SignalProcessingChain/DIS
- U15 pad 4: /PerCoil/SignalProcessingChain/HEN -> GND
- U15 pad 5: +5V -> /PerCoil/SignalProcessingChain/Out
- U15 pad 6: /C1 -> /PerCoil/SignalProcessingChain/DIR
- U17 pad 1: Net-(D8-K) -> Net-(U17A-+)
- U17 pad 2: /PerCoil/SignalProcessingChain/HEN -> /Vtri
- U17 pad 3: /PerCoil/SignalProcessingChain/DIS -> Net-(U17B-+)
- U17 pad 4: GND -> /Vtri
- U17 pad 5: /PerCoil/SignalProcessingChain/Out -> GND
- U17 pad 6: /PerCoil/SignalProcessingChain/DIR -> /PerCoil1/SignalProcessingChain/HF PWM
- U17 pad 7: /VCM -> /PerCoil/SignalProcessingChain/HF PWM
- U17 pad 8: Net-(U17-HDEL) -> +5V
- U18 pad 1: /PerCoil/AH -> Net-(U18A-+)
- U18 pad 2: VBUS -> /PerCoil/OC_SENSE
- U18 pad 3: /+OUT1 -> Net-(U18B-+)
- U18 pad 4: /PerCoil/AL -> Net-(U18B--)
- U18 pad 5: /PerCoil/OC_SENSE -> GND
- U18 pad 6: /PerCoil/OC_SENSE -> /PerCoil/SignalProcessingChain/Current_Dir
- U18 pad 7: /PerCoil/BL -> /PerCoil/~{OC1}
- U18 pad 8: /PerCoil/BHS -> +5V
- U20 pad 1: /PerCoil1/AH -> /A1
- U20 pad 2: VBUS -> Net-(U18B-+)
- U20 pad 3: /+OUT2 -> /VCM
- U21 pad 1: Net-(U21--) -> /A1
- U21 pad 2: GND -> Net-(U18B--)
- U21 pad 3: GND -> /VCM
- U22 pad 1: Net-(U22A-+) -> /PerCoil/AH
- U22 pad 2: /PerCoil1/SignalProcessingChain/Vtri -> Vdrive
- U22 pad 3: Net-(U22B-+) -> /+OUT1
- U22 pad 4: /PerCoil1/SignalProcessingChain/Vtri -> /PerCoil/AL
- U22 pad 5: GND -> /PerCoil/OC_SENSE
- U22 pad 6: /PerCoil1/SignalProcessingChain/HF PWM -> /PerCoil/OC_SENSE
- U22 pad 7: /PerCoil1/SignalProcessingChain/Vsq -> /PerCoil/BL
- U22 pad 8: +5V -> /PerCoil/BHS
- U23 pad 1: /PerCoil1/SignalProcessingChain/HF PWM -> Net-(U23--)
- U23 pad 3: /PWM4 -> GND
- U23 pad 4: Net-(U23-Z) -> GND
- U23 pad 5: +5V -> Net-(R23-Pad2)
- U23 pad 6: /B2 -> +5V
- U26 pad 1: +5V -> Net-(U26A-+)
- U26 pad 2: GND -> Net-(U26A--)
- U26 pad 3: Net-(U25-Z) -> Net-(U26B-+)
- U26 pad 4: /PerCoil1/SignalProcessingChain/HEN -> /PerCoil1/OC_SENSE
- U26 pad 5: +5V -> GND
- U26 pad 6: /C2 -> /PerCoil1/~{OC1}
- U28 pad 1: Net-(D12-K) -> /A2
- U28 pad 2: /PerCoil1/SignalProcessingChain/HEN -> Net-(U26A-+)
- U28 pad 3: /PerCoil1/SignalProcessingChain/DIS -> /VCM
- U29 pad 1: Net-(U29A--) -> /A2
- U29 pad 2: Net-(U29A--) -> Net-(U26A--)
- U29 pad 3: Net-(U29A-+) -> /VCM
- U30 pad 1: Net-(U30-K) -> /PerCoil1/AH
- U30 pad 2: Net-(U30-K) -> Vdrive
- U30 pad 3: GND -> /+OUT2
- U5 pad 1: Net-(U3-Z) -> Net-(U5A-+)
- U5 pad 2: GND -> /Vtri
- U5 pad 3: Net-(U4-Z) -> GND
- U5 pad 4: Net-(U5-Z) -> GND
- U5 pad 5: +5V -> GND
- U5 pad 6: Net-(D3-K) -> unconnected-(U5-Pad6)
- U6 pad 1: /EN1 -> Net-(U3-Z)
- U6 pad 2: /~{OC1} -> GND
- U6 pad 3: /PerCoil/EN -> Net-(U4-Z)
- U6 pad 4: /EN2 -> Net-(U6-Z)
- U6 pad 5: /~{OC2} -> +5V
- U6 pad 6: /PerCoil1/EN -> Net-(D4-K)
- U7 pad 8: Net-(U5-Z) -> Net-(U6-Z)
- U8 pad 1: Net-(U8A-+) -> /PerCoil/SignalProcessingChain/HF PWM
- U8 pad 2: /PerCoil/OC_SENSE -> GND
- U8 pad 3: Net-(U8B-+) -> /PWM2
- U8 pad 4: /PerCoil1/OC_SENSE -> Net-(U11-I0)
- U8 pad 5: GND -> +5V
- U8 pad 6: /~{OC2} -> /B1
- U9 pad 1: /~{OC1} -> /PerCoil/SignalProcessingChain/HF PWM
- U9 pad 2: Net-(R13-Pad2) -> GND
- U9 pad 3: /~{OC2} -> /PWM1
- U9 pad 4: Net-(R14-Pad2) -> Net-(U10-I1)
- U9 pad 5: /PerCoil/EN -> +5V
- U9 pad 6: Net-(U16-I0) -> /A1
Routing:
- net +5V: track 0.00 -> 33.9 mm
- net GND: track 0.00 -> 29.8 mm
- net +12V: track 0.00 -> 25.8 mm, vias 0 -> 2
- net /A1: track 0.00 -> 23.1 mm
- net Net-(U18B-+): track 0.00 -> 19.7 mm
- net /-OUT1: track 0.00 -> 16.7 mm
- net /PerCoil/SignalProcessingChain/EN: track 0.00 -> 15.6 mm, vias 0 -> 2
- net Net-(U23--): track 0.00 -> 13.6 mm
- net Net-(U18B--): track 0.00 -> 12.9 mm
- net /VCM: track 0.00 -> 8.81 mm
- net /PerCoil/SignalProcessingChain/HEN: track 0.00 -> 8.25 mm
- net Net-(U13-Z): track 0.00 -> 6.72 mm
- net Net-(D6-K): track 0.00 -> 6.49 mm
- net Net-(D7-K): track 0.00 -> 6.47 mm
- net /C1: track 0.00 -> 6.43 mm, vias 0 -> 2
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
Commit message: saving here before i try making PerCoilFlipped on schematic
Parts:
- removed C20, C21, C37, C38: 2.2u, Capacitor_SMD:C_0603_1608Metric
- removed D4, D5: D_logic, Diode_SMD:D_SMA
- removed R9: 10k, Resistor_SMD:R_0603_1608Metric
- added U16: NC7SZ157P6X, Package_TO_SOT_SMD:SOT-363_SC-70-6, F.Cu at (84.3, 165.8)
- A1: footprint Module:Arduino_UNO_R3_ConnOnly -> Module:Arduino_UNO_R3_ConnOnly_Coil_Driver; moved to B.Cu
- TP1, TP3: moved to B.Cu
- U7: footprint Package_SON:WSON-10-1EP_3x3mm_P0.5mm_EP1.6x2mm -> Package_SON:WSON-10-1_3x3mm_P0.5mm_1.6x2mm
- moved C34 193.4 mm to (214.5, 145.4), turned to -90 degrees
- moved A1 169.1 mm to (99.6, 123.5), turned to 180 degrees
- moved U3 165.4 mm to (79.3, 165.8)
- moved U4 164.6 mm to (79.3, 168.8)
- moved C39 163.9 mm to (86.8, 168.8), turned to -90 degrees
- moved C40 163.4 mm to (81.8, 168.9), turned to -90 degrees
- moved U6 158.7 mm to (84.3, 168.8)
- moved C41 158.3 mm to (81.8, 165.7), turned to 90 degrees
- moved U7 158.0 mm to (89.2, 166.7), turned to -90 degrees
- moved R1 155.9 mm to (62.5, 173.7)
- moved TP1 154.0 mm to (89.2, 166.8), turned to 180 degrees
- moved C42 153.8 mm to (86.8, 165.7), turned to 90 degrees
- moved U2 148.5 mm to (63.5, 169.1), turned to -90 degrees
- moved R5 135.8 mm to (103.3, 126.5), turned to 90 degrees
- moved D2 128.1 mm to (94.7, 135.9), turned to 90 degrees
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Connections:
- C19 pad 1: Net-(U17B-+) -> Net-(U17B--)
- C5 pad 1: Net-(U17A-+) -> Net-(U17A--)
- D10 pad 2: Net-(D10-A) -> +5V
- D2 pad 2: Net-(D2-A) -> VBUS
- D8 pad 2: Net-(D8-A) -> +5V
- J1 pad A9: Net-(D2-A) -> VBUS
- J1 pad B9: Net-(D2-A) -> VBUS
- R10 pad 2: Net-(U17A-+) -> Net-(U17A--)
- R11 pad 1: Net-(U17A-+) -> Net-(U17A--)
- R12 pad 2: Net-(U17A-+) -> Net-(U17A--)
- R19 pad 1: Net-(D8-A) -> Net-(U14D-Y)
- R19 pad 2: +5V -> Net-(D8-K)
- R25 pad 1: Net-(U26B-+) -> Net-(U26A-+)
- R27 pad 2: Net-(U26B-+) -> Net-(U26A-+)
- R28 pad 1: Net-(D10-A) -> Net-(U38D-Y)
- R28 pad 2: +5V -> Net-(D10-K)
- R34 pad 2: Net-(U17B-+) -> Net-(U17B--)
- R35 pad 1: Net-(U17B-+) -> Net-(U17B--)
- R36 pad 2: Net-(U17B-+) -> Net-(U17B--)
- U14 pad 13: Net-(D8-K) -> Net-(U14D-Y)
- U17 pad 1: Net-(U17A-+) -> /Vtri
- U17 pad 2: /Vtri -> Net-(U17A--)
- U17 pad 3: Net-(U17B-+) -> /Vtri
- U17 pad 4: /Vtri -> Net-(U17B--)
- U26 pad 2: Net-(U26A--) -> /PerCoil1/OC_SENSE
- U26 pad 4: /PerCoil1/OC_SENSE -> Net-(U26B--)
- U26 pad 6: /PerCoil1/~{OC1} -> /PerCoil1/SignalProcessingChain/Current_Dir
- U26 pad 7: /PerCoil1/SignalProcessingChain/Current_Dir -> /PerCoil1/~{OC1}
- U28 pad 2: Net-(U26A-+) -> Net-(U26B-+)
- U29 pad 2: Net-(U26A--) -> Net-(U26B--)
- U38 pad 13: Net-(D10-K) -> Net-(U38D-Y)
Routing:
- net +5V: track 33.9 -> 106.1 mm, vias 0 -> 2
- net GND: track 29.8 -> 87.0 mm
- net +12V: track 25.8 -> 60.4 mm, vias 2 -> 4
- net /Vtri: track 0.00 -> 32.0 mm
- net /PerCoil/SignalProcessingChain/HF PWM: track 4.25 -> 23.5 mm
- net VBUS: track 0.00 -> 14.9 mm
- net /PerCoil/SignalProcessingChain/Current_Dir: track 0.00 -> 14.5 mm, vias 0 -> 2
- net /PerCoil/SignalProcessingChain/DIS: track 5.97 -> 19.8 mm, vias 0 -> 2
- net /DACOUT2: track 0.00 -> 12.4 mm, vias 0 -> 2
- net /VCM: track 8.81 -> 19.8 mm
- net /Vsq: track 0.00 -> 9.17 mm
- net Net-(J1-CC1): track 0.00 -> 8.35 mm
- net Net-(J1-CC2): track 0.00 -> 8.19 mm
- net Net-(U40A-+): track 0.00 -> 7.85 mm
- net Net-(D12-K): track 0.00 -> 6.85 mm
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
Commit message: Fixed schematic after annotation fuck up
Connections:
- C19 pad 1: Net-(U17B--) -> Net-(U17B-+)
- C5 pad 1: Net-(U17A--) -> Net-(U17A-+)
- D10 pad 2: +5V -> Net-(D10-A)
- D8 pad 2: +5V -> Net-(D8-A)
- R10 pad 2: Net-(U17A--) -> Net-(U17A-+)
- R11 pad 1: Net-(U17A--) -> Net-(U17A-+)
- R12 pad 2: Net-(U17A--) -> Net-(U17A-+)
- R19 pad 1: Net-(U14D-Y) -> Net-(D8-A)
- R19 pad 2: Net-(D8-K) -> +5V
- R25 pad 1: Net-(U26A-+) -> Net-(U26B-+)
- R27 pad 2: Net-(U26A-+) -> Net-(U26B-+)
- R28 pad 1: Net-(U38D-Y) -> Net-(D10-A)
- R28 pad 2: Net-(D10-K) -> +5V
- R34 pad 2: Net-(U17B--) -> Net-(U17B-+)
- R35 pad 1: Net-(U17B--) -> Net-(U17B-+)
- R36 pad 2: Net-(U17B--) -> Net-(U17B-+)
- U14 pad 13: Net-(U14D-Y) -> Net-(D8-K)
- U17 pad 1: /Vtri -> Net-(U17A-+)
- U17 pad 2: Net-(U17A--) -> /Vtri
- U17 pad 3: /Vtri -> Net-(U17B-+)
- U17 pad 4: Net-(U17B--) -> /Vtri
- U26 pad 2: /PerCoil1/OC_SENSE -> Net-(U26A--)
- U26 pad 4: Net-(U26B--) -> /PerCoil1/OC_SENSE
- U26 pad 6: /PerCoil1/SignalProcessingChain/Current_Dir -> /PerCoil1/~{OC1}
- U26 pad 7: /PerCoil1/~{OC1} -> /PerCoil1/SignalProcessingChain/Current_Dir
- U28 pad 2: Net-(U26B-+) -> Net-(U26A-+)
- U29 pad 2: Net-(U26B--) -> Net-(U26A--)
- U38 pad 13: Net-(U38D-Y) -> Net-(D10-K)
Routing:
- net /Vtri: track 32.0 -> 12.9 mm
- net Net-(U17B-+): track 0.00 -> 10.3 mm
- net Net-(U17A-+): track 0.00 -> 8.86 mm
- net Net-(U14D-Y): track 2.20 -> 0.00 mm
- net Net-(D8-K): track 2.23 -> 4.43 mm
